Commit message: working demo with gui

File: robot_arm_description_urdfv6/urdf/robot_arm_description_urdfv6.urdf (robot description, URDF)
Before this commit: robot robot_arm_description_urdfv6, 9 links, 8 joints
Joints:
- joint grip_fixed: origin xyz=-0.060 0.097 0.0285 rpy=1.5708 1.5708 0 -> xyz=-0.060 0.097 0.0285 rpy=-1.5708 0 0
- joint joint1: axis 0 0 1 -> 0 0 -1
- joint joint5: limit lower=-2.61 upper=0 effort=0 velocity=0 -> lower=0 upper=2.61 effort=0 velocity=0

File: robot_arm_moveit_config/config/gazebo_robot_arm_description_urdfv6.urdf (robot description, URDF)
Before this commit: robot robot_arm_description_urdfv6, 9 links, 8 joints
Joints:
- joint grip_fixed: origin xyz=-0.060 0.097 0.0285 rpy=1.5708 1.5708 0 -> xyz=-0.060 0.097 0.0285 rpy=-1.5708 0 0
