Commit message: camera and unfixed bugs

File: robot_arm_moveit_config/config/gazebo_robot_arm_description_urdfv6.urdf (robot description, URDF)
Before this commit: robot robot_arm_description_urdfv6, 9 links, 8 joints
Joints:
- joint joint1: axis 0 0 1 -> 0 0 -1
- joint joint5: limit lower=-2.61 upper=0 effort=0 velocity=0 -> lower=0 upper=2.61 effort=0 velocity=0
